Commit message: Arthur got xacro version for multiple drones working.

File: urdf/drone_base.urdf.xacro (robot description, xacro)
@@ -1,6 +1,5 @@
 <?xml version="1.0"?>
 <robot xmlns:xacro="http://www.ros.org/wiki/xacro">
-  <xacro:macro name="drone_base" params="prefix">
-    <link name="${prefix}base_link" />
+  <xacro:macro name="drone_base" params="prefix base_link_name">
     <link name="${prefix}x" />
     <link name="${prefix}xy" />
@@ -8,5 +7,5 @@
     <link name="${prefix}mobile" />
     <joint name="${prefix}move_x" type="prismatic" >
-      <parent link="${prefix}base_link" />
+      <parent link="${base_link_name}" />
       <child link="${prefix}x" />
       <axis xyz="1 0 0" />

File: urdf/multi_drones.urdf.xacro (robot description, xacro)
@@ -3,4 +3,6 @@
   <xacro:include filename="$(find aapacs_drones)/urdf/drone_base.urdf.xacro" />
   <link name="base_link" />
-  <xacro:drone_base prefix="" base_link_name="base_link" />
+  <xacro:drone_base prefix="drone1_" base_link_name="base_link" />
+  <xacro:drone_base prefix="drone2_" base_link_name="base_link" />
+  <xacro:drone_base prefix="drone3_" base_link_name="base_link" />
 </robot>

File: urdf/two_drones.urdf.xacro (robot description, xacro)
@@ -3,4 +3,5 @@
   <xacro:include filename="$(find aapacs_drones)/urdf/drone_base.urdf.xacro" />
   <link name="base_link" />
-  <xacro:drone_base prefix="" base_link_name="base_link" />
+  <xacro:drone_base prefix="drone3_" base_link_name="base_link" />
+  <xacro:drone_base prefix="drone2_" base_link_name="base_link" />
 </robot>

Commit message: Arthur fixed a few fuerte things and combined the drone visualization with the xacro URDF.

File: urdf/drone_base.urdf.xacro (robot description, xacro)
@@ -5,5 +5,21 @@
     <link name="${prefix}xy" />
     <link name="${prefix}xyz" />
-    <link name="${prefix}mobile" />
+    <link name="${prefix}hull">
+      <visual>
+        <geometry>
+          <box size="0.5 0.5 0.05"/>
+        </geometry>
+        <origin xyz="0 0 0.1"/>
+        <material name="${prefix}hull_color">
+          <color rgba="0.5 0.5 0.5 1"/>
+        </material>
+      </visual>
+      <collision>
+        <geometry>
+          <box size="0.5 0.5 0.2"/>
+        </geometry>
+        <origin xyz="0 0 0.1"/>
+      </collision>
+    </link>
     <joint name="${prefix}move_x" type="prismatic" >
       <parent link="${base_link_name}" />
@@ -26,8 +42,64 @@
     <joint name="${prefix}turn_z" type="revolute" >
       <parent link="${prefix}xyz" />
-      <child link="${prefix}mobile" />
+      <child link="${prefix}hull" />
       <axis xyz="0 0 1" />
       <limit lower="-3.141" upper="3.141" effort="100" velocity="100" />
     </joint>
+  <link name="${prefix}fr_rotor">
+    <visual>
+      <geometry>
+        <cylinder radius="0.12" length="0.06"/>
+      </geometry>
+      <origin xyz="0.125 0.125 0.1"/>
+      <material name="${prefix}front_rotor_color">
+        <color rgba="0.8 0.4 0.4 1"/>
+      </material>
+    </visual>
+  </link>
+  <joint name="${prefix}fr_rotor_joint" type="fixed">
+    <parent link="${prefix}hull"/>
+    <child link="${prefix}fr_rotor"/>
+  </joint>
+  <link name="${prefix}fl_rotor">
+    <visual>
+      <geometry>
+        <cylinder radius="0.12" length="0.06"/>
+      </geometry>
+      <origin xyz="0.125 -0.125 0.1"/>
+      <material name="${prefix}front_rotor_color"/>
+    </visual>
+  </link>
+  <joint name="${prefix}fl_rotor_joint" type="fixed">
+    <parent link="${prefix}hull"/>
+    <child link="${prefix}fl_rotor"/>
+  </joint>
+  <link name="${prefix}br_rotor">
+    <visual>
+      <geometry>
+        <cylinder radius="0.12" length="0.06"/>
+      </geometry>
+      <origin xyz="-0.125 0.125 0.1"/>
+      <material name="${prefix}back_rotor_color">
+        <color rgba="0.4 0.4 0.4 1"/>
+      </material>
+    </visual>
+  </link>
+  <joint name="${prefix}br_rotor_joint" type="fixed">
+    <parent link="${prefix}hull"/>
+    <child link="${prefix}br_rotor"/>
+  </joint>
+  <link name="${prefix}bl_rotor">
+    <visual>
+      <geometry>
+        <cylinder radius="0.12" length="0.06"/>
+      </geometry>
+      <origin xyz="-0.125 -0.125 0.1"/>
+      <material name="${prefix}back_rotor_color"/>
+    </visual>
+  </link>
+  <joint name="${prefix}bl_rotor_joint" type="fixed">
+    <parent link="${prefix}hull"/>
+    <child link="${prefix}bl_rotor"/>
+  </joint>
   </xacro:macro>
 </robot>
